Commit message: all_legs following first

File: urdf/auto.urdf (robot description, URDF)
Before this commit: robot me, 10 links, 9 joints
Joints:
- joint rota_3: origin xyz=-5 5 0 rpy=-1.57 0 3.14 -> xyz=-5 -5 0 rpy=-1.57 0 3.14
- joint rota_4: origin xyz=-5 -5 0 rpy=-1.57 0 3.14 -> xyz=-5 5 0 rpy=-1.57 0 3.14

File: urdf/quadra.xacro (robot description, xacro)
@@ -92,8 +92,8 @@
     </xacro:leg>
     <xacro:leg leg_no='3'>
+        <origin xyz="-5 -5 0" rpy="-1.57 0 3.14"/>
+    </xacro:leg>
+    <xacro:leg leg_no='4'>
         <origin xyz="-5 5 0" rpy="-1.57 0 3.14"/>
     </xacro:leg>
-    <xacro:leg leg_no='4'>
-        <origin xyz="-5 -5 0" rpy="-1.57 0 3.14"/>
-    </xacro:leg>
 </robot>
