Commit message: everythong working noise in rviz

File: urdf/ele.xacro (robot description, xacro)
@@ -3,4 +3,5 @@
     <!-- Xacro defn for a leg -->
     <xacro:macro name="leg" params="leg_no *origin">
+        <!-- Joints -->
         <joint name="hip_${leg_no}" type="continuous">
             <parent link="chassis"/>
@@ -23,4 +24,33 @@
             <origin xyz="4 0 0" rpy="0 0 0"/>
         </joint>
+        <!-- Transmissions -->
+        <transmission name="hip_trans_${leg_no}">
+            <type>transmission_interface/SimpleTransmission</type>
+            <actuator name="hip_motor_${leg_no}">
+            <mechanicalReduction>1</mechanicalReduction>
+            </actuator>
+            <joint name="hip_${leg_no}">
+            <hardwareInterface>hardware_interface/PositionJointInterface</hardwareInterface>
+            </joint>
+        </transmission>
+        <transmission name="knee_trans_${leg_no}">
+            <type>transmission_interface/SimpleTransmission</type>
+            <actuator name="knee_motor_${leg_no}">
+            <mechanicalReduction>1</mechanicalReduction>
+            </actuator>
+            <joint name="knee_${leg_no}">
+            <hardwareInterface>hardware_interface/PositionJointInterface</hardwareInterface>
+            </joint>
+        </transmission>
+        <transmission name="ankle_trans_${leg_no}">
+            <type>transmission_interface/SimpleTransmission</type>
+            <actuator name="ankle_motor_${leg_no}">
+            <mechanicalReduction>1</mechanicalReduction>
+            </actuator>
+            <joint name="ankle_${leg_no}">
+            <hardwareInterface>hardware_interface/PositionJointInterface</hardwareInterface>
+            </joint>
+        </transmission>
+        <!-- Links -->
         <link name="thigh_${leg_no}">
             <collision>
@@ -128,3 +158,8 @@
         <origin xyz="5 0 -5" rpy="0 0 0"/>
     </xacro:leg>
+    <gazebo>
+        <plugin name="gazebo_ros_control" filename="libgazebo_ros_control.so">
+        <robotNamespace>/</robotNamespace>
+        </plugin>
+    </gazebo>
 </robot>

Commit message: matlab added with one link

File: urdf/ele.xacro (robot description, xacro)
@@ -9,4 +9,5 @@
             <axis xyz="0 0 1"/>
             <xacro:insert_block name="origin" />
+            <limit effort="5" velocity="1.0" lower="-3.14159" upper="3.14159"/>
         </joint>
         <joint name="knee_${leg_no}" type="revolute">
@@ -14,5 +15,6 @@
             <child link="calf_${leg_no}"/>
             <axis xyz="0 0 1"/>
-            <limit lower="-3.14159" upper="3.14159" velocity="50.0" effort="1000.0"/>
+            <!-- <limit lower="-3.14159" upper="3.14159" velocity="50.0" effort="1000.0"/> -->
+            <limit effort="5" velocity="1.0" lower="-3.14159" upper="3.14159"/>
             <origin xyz="6 0 0" rpy="0 0 0"/>
         </joint>
@@ -21,5 +23,5 @@
             <child link="foot_${leg_no}"/>
             <axis xyz="0 0 1"/>
-            <limit lower="-3.14159" upper="3.14159" velocity="50.0" effort="1000.0"/>
+            <limit effort="5" velocity="1.0" lower="-3.14159" upper="3.14159"/>
             <origin xyz="4 0 0" rpy="0 0 0"/>
         </joint>
@@ -119,4 +121,11 @@
             </inertial>
         </link>
+        <gazebo reference="foot_${leg_no}">
+            <mu1 value="200.0"/>
+            <mu2 value="100.0"/>
+            <kp value="10000000.0" />
+            <kd value="1.0" />
+            <material>Gazebo/Grey</material>
+        </gazebo>
     </xacro:macro>
     <!-- fixed frame and link without xacro -->
@@ -141,6 +150,6 @@
         </visual>
         <inertial>
-            <mass value="10"/>
-            <inertia ixx="1" ixy="0" ixz="0" iyy="1" iyz="0" izz="1"/>
+            <mass value="1000"/>
+            <inertia ixx="100" ixy="0" ixz="0" iyy="100" iyz="0" izz="100"/>
         </inertial>
     </link>
