Commit message: fd_mv _dwn working trajectroy not corrected

File: urdf/ele.urdf (robot description, URDF)
Before this commit: robot me, 5 links, 4 joints
Joints:
- joint ankle_1: origin xyz=0 -4 0 rpy=0 0 0 -> xyz=4 0 0 rpy=0 0 0
- joint knee_1: origin xyz=0 -6 0 rpy=0 0 0 -> xyz=6 0 0 rpy=0 0 0

File: urdf/ele.xacro (robot description, xacro)
@@ -14,5 +14,5 @@
             <axis xyz="0 0 1"/>
             <limit lower="-3.14159" upper="3.14159" velocity="50.0" effort="1000.0"/>
-            <origin xyz="0 -6 0" rpy="0 0 0"/>
+            <origin xyz="6 0 0" rpy="0 0 0"/>
         </joint>
         <joint name="ankle_${leg_no}" type="revolute">
@@ -21,9 +21,9 @@
             <axis xyz="0 0 1"/>
             <limit lower="-3.14159" upper="3.14159" velocity="50.0" effort="1000.0"/>
-            <origin xyz="0 -4 0" rpy="0 0 0"/>
+            <origin xyz="4 0 0" rpy="0 0 0"/>
         </joint>
         <link name="thigh_${leg_no}">
             <collision>
-                <origin xyz="0.0 -3 0" rpy="1.57 0.0 0.0"/>
+                <origin xyz="3 0 0" rpy="0 1.57 0"/>
                 <geometry>
                     <cylinder radius="0.25" length="6"/>
@@ -31,5 +31,5 @@
             </collision>
             <visual>
-                <origin xyz="0.0 -3 0" rpy="1.57 0.0 0"/>
+                <origin xyz="3 0 0" rpy="0 1.57 0"/>
                 <geometry>
                     <cylinder radius="0.25" length="6"/>
@@ -43,5 +43,5 @@
         <link name="calf_${leg_no}">
             <collision>
-                <origin xyz="0.0 -2 0.0" rpy="1.57 0.0 0.0"/>
+                <origin xyz="2 0 0.0" rpy="0 1.57 0.0"/>
                 <geometry>
                     <cylinder radius="0.25" length="4"/>
@@ -49,5 +49,5 @@
             </collision>
             <visual>
-                <origin xyz="0.0 -2 0.0" rpy="1.57 0.0 0.0"/>
+                <origin xyz="2 0 0.0" rpy="0 1.57 0.0"/>
                 <geometry>
                     <cylinder radius="0.25" length="4"/>
@@ -67,5 +67,5 @@
         <link name="foot_${leg_no}">
             <collision>
-                <origin xyz="0.0 -1 0.0" rpy="1.57 0.0 0.0"/>
+                <origin xyz="1 0 0.0" rpy="0.0 1.57 0.0"/>
                 <geometry>
                     <cylinder radius="0.25" length="2"/>
@@ -73,5 +73,5 @@
             </collision>
             <visual>
-                <origin xyz="0.0 -1 0.0" rpy="1.57 0.0 0.0"/>
+                <origin xyz="1 0 0.0" rpy="0.0 1.57 0.0"/>
                 <geometry>
                     <cylinder radius="0.25" length="2"/>

Commit message: Working Unknown bug in mv dwn

File: urdf/ele.urdf (robot description, URDF)
Before this commit: robot me, 5 links, 4 joints
Links:
- added link calf_2, mass 10; collision cylinder length=4 radius=0.25; visual cylinder length=4 radius=0.25
- added link calf_3, mass 10; collision cylinder length=4 radius=0.25; visual cylinder length=4 radius=0.25
- added link calf_4, mass 10; collision cylinder length=4 radius=0.25; visual cylinder length=4 radius=0.25
- added link foot_2, mass 10; collision cylinder length=2 radius=0.25; visual cylinder length=2 radius=0.25
- added link foot_3, mass 10; collision cylinder length=2 radius=0.25; visual cylinder length=2 radius=0.25
- added link foot_4, mass 10; collision cylinder length=2 radius=0.25; visual cylinder length=2 radius=0.25
- added link thigh_2, mass 10; collision cylinder length=6 radius=0.25; visual cylinder length=6 radius=0.25
- added link thigh_3, mass 10; collision cylinder length=6 radius=0.25; visual cylinder length=6 radius=0.25
- added link thigh_4, mass 10; collision cylinder length=6 radius=0.25; visual cylinder length=6 radius=0.25
Joints:
- added joint ankle_2: type revolute, parent calf_2, child foot_2, origin xyz=4 0 0 rpy=0 0 0, axis 0 0 1, limit lower=-3.14159 upper=3.14159 effort=1000.0 velocity=50.0
- added joint ankle_3: type revolute, parent calf_3, child foot_3, origin xyz=4 0 0 rpy=0 0 0, axis 0 0 1, limit lower=-3.14159 upper=3.14159 effort=1000.0 velocity=50.0
- added joint ankle_4: type revolute, parent calf_4, child foot_4, origin xyz=4 0 0 rpy=0 0 0, axis 0 0 1, limit lower=-3.14159 upper=3.14159 effort=1000.0 velocity=50.0
- added joint hip_2: type continuous, parent chassis, child thigh_2, origin xyz=5 0 5 rpy=0 0 0, axis 0 0 1
- added joint hip_3: type continuous, parent chassis, child thigh_3, origin xyz=-5 0 -5 rpy=0 0 0, axis 0 0 1
- added joint hip_4: type continuous, parent chassis, child thigh_4, origin xyz=5 0 -5 rpy=0 0 0, axis 0 0 1
- added joint knee_2: type revolute, parent thigh_2, child calf_2, origin xyz=6 0 0 rpy=0 0 0, axis 0 0 1, limit lower=-3.14159 upper=3.14159 effort=1000.0 velocity=50.0
- added joint knee_3: type revolute, parent thigh_3, child calf_3, origin xyz=6 0 0 rpy=0 0 0, axis 0 0 1, limit lower=-3.14159 upper=3.14159 effort=1000.0 velocity=50.0
- added joint knee_4: type revolute, parent thigh_4, child calf_4, origin xyz=6 0 0 rpy=0 0 0, axis 0 0 1, limit lower=-3.14159 upper=3.14159 effort=1000.0 velocity=50.0

File: urdf/ele.xacro (robot description, xacro)
@@ -2,5 +2,5 @@
 <robot xmlns:xacro="http://www.ros.org/wiki/xacro" name="me">
     <!-- Xacro defn for a leg -->
-    <xacro:macro name="hind_leg" params="leg_no *origin">
+    <xacro:macro name="leg" params="leg_no *origin">
         <joint name="hip_${leg_no}" type="continuous">
             <parent link="chassis"/>
@@ -116,15 +116,15 @@
     </link>
     <!-- leg links with xacro -->
-    <xacro:hind_leg leg_no='1'>
+    <xacro:leg leg_no='1'>
         <origin xyz="-5 0 5" rpy="0 0 0"/>
-    </xacro:hind_leg>
-    <!-- <xacro:leg leg_no='2'>
-        <origin xyz="5 -5 0" rpy="-1.57 0 3.14"/>
+    </xacro:leg>
+    <xacro:leg leg_no='2'>
+        <origin xyz="5 0 5" rpy="0 0 0"/>
     </xacro:leg>
     <xacro:leg leg_no='3'>
-        <origin xyz="-5 -5 0" rpy="-1.57 0 3.14"/>
+        <origin xyz="-5 0 -5" rpy="0 0 0"/>
     </xacro:leg>
     <xacro:leg leg_no='4'>
-        <origin xyz="-5 5 0" rpy="-1.57 0 3.14"/>
-    </xacro:leg> -->
+        <origin xyz="5 0 -5" rpy="0 0 0"/>
+    </xacro:leg>
 </robot>

Commit message: matlab ik working

File: urdf/ele.urdf (robot description, URDF)
Before this commit: robot me, 14 links, 13 joints
Links:
- removed link calf_2
- removed link calf_3
- removed link calf_4
- removed link foot_2
- removed link foot_3
- removed link foot_4
- removed link thigh_2
- removed link thigh_3
- removed link thigh_4
- link chassis: mass 10 -> 1000
Joints:
- removed joint ankle_2
- removed joint ankle_3
- removed joint ankle_4
- removed joint hip_2
- removed joint hip_3
- removed joint hip_4
- removed joint knee_2
- removed joint knee_3
- removed joint knee_4
- joint ankle_1: limit lower=-3.14159 upper=3.14159 effort=1000.0 velocity=50.0 -> lower=-3.14159 upper=3.14159 effort=5 velocity=1.0
- joint hip_1: limit (none) -> lower=-3.14159 upper=3.14159 effort=5 velocity=1.0
- joint knee_1: limit lower=-3.14159 upper=3.14159 effort=1000.0 velocity=50.0 -> lower=-3.14159 upper=3.14159 effort=5 velocity=1.0

File: urdf/ele.xacro (robot description, xacro)
@@ -158,5 +158,5 @@
         <origin xyz="-5 0 5" rpy="0 0 0"/>
     </xacro:leg>
-    <xacro:leg leg_no='2'>
+    <!-- <xacro:leg leg_no='2'>
         <origin xyz="5 0 5" rpy="0 0 0"/>
     </xacro:leg>
@@ -166,5 +166,5 @@
     <xacro:leg leg_no='4'>
         <origin xyz="5 0 -5" rpy="0 0 0"/>
-    </xacro:leg>
+    </xacro:leg> -->
     <gazebo>
         <plugin name="gazebo_ros_control" filename="libgazebo_ros_control.so">
